File: Hardware/pcbusinesscard.kicad_pcb (KiCad board)
At the start: 4 copper layers, 89 x 51 mm, 104 parts, among them J10 USB_C_Receptacle_USB2.0, J2 Micro_SD_Card, J4 Conn_01x03, J5 Conn_ST_STDC14, J6 Conn_01x04_Pin, J7 Conn_01x04_Pin, Q1 MMBT3904, Q2 MMBT3904, Q3 MMBT3904, Q4 MMBT3904, Q5 MMBT3904, SW1 ESC, SW3 1, SW4 2, SW5 SW_Nidec_CAS-120A1, SW98 SW_Push, U1 RP2040, U10 NRF24L01, U12 LM2596S-3.3, U2 24AA025E-OT, U3 24AA025E-OT, U4 24AA025E-OT, U5 BQ24090DGQ, U8 MCP1700x-330xxTT, U9 TPS2116DRL, Y1 12MHz, Y2 Crystal

Commit message: dont remember
Other:
- board text added: "647 XXX XXXX"
- board text added: "Aryan Ghosh"
- board text added: "aryan.ghosh@mail.utoronto.ca"
- board text added: "github.com/Aryan-G4"
- board text added: "linkedin.com/in/aryan-gh0sh"

Commit message: Fixed DRC and cleaned up schematic
Parts:
- moved C16 0.20 mm to (90.5, 51.2)
- moved TP5 0.20 mm to (97.6, 60.4)
Routing:
- net GND: track 181.1 -> 185.6 mm, vias 98 -> 97
- net /RP_I2C1_SCL: track 113.0 -> 115.5 mm
- net /RP_I2C1_SDA: track 109.3 -> 110.8 mm
